File: Solar_Battery.kicad_sch (KiCad schematic)
At the start: 0 parts

Commit message: Finished Rectifier Organization
Changed lines of the file:
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@@
 			(width 0.1524)
 			(type solid)
+			(color 0 89 255 1)
 		)
 		(fill
-			(color 0 0 0 0)
+			(color 0 64 255 0.5019607843)
 		)
 		(property "Sheetname" "Battery_Controller"
 			(at 156.21 75.4884 0)
-			(show_name yes)
+			(show_name no)
 			(do_not_autoplace no)
 			(effects
 				(font
 					(size 1.27 1.27)
+					(thickness 0.254)
+					(bold yes)
 				)
 				(justify left bottom)
@@
 		(property "Sheetfile" "Battery_Controller.kicad_sch"
 			(at 156.21 117.4246 0)
-			(show_name yes)
+			(hide yes)
+			(show_name no)
 			(do_not_autoplace no)
 			(effects
@@
 		(on_board yes)
 		(dnp no)
-		(fields_autoplaced yes)
 		(stroke
 			(width 0.1524)
 			(type solid)
+			(color 45 255 131 1)
 		)
 		(fill
-			(color 0 0 0 0)
+			(color 70 255 92 0.3019607843)
 		)
 		(property "Sheetname" "Rectifier"
-			(at 97.79 75.4884 0)
+			(at 98.044 75.692 0)
 			(show_name no)
 			(do_not_autoplace no)
@@
 				(font
 					(size 1.27 1.27)
+					(thickness 0.254)
+					(bold yes)
 				)
 				(justify left bottom)
@@
 		(property "Sheetfile" "Rectifier.kicad_sch"
 			(at 97.79 117.4246 0)
+			(hide yes)
 			(show_name no)
 			(do_not_autoplace no)
