File: Rectifier.kicad_sch (KiCad schematic)
At the start: 0 parts

Commit message: Finished Rectifier Organization
Other:
- added sheet Transformer_Output (Transformer_Output.kicad_sch)
- added sheet UCC_Chip (UCC_Chip.kicad_sch)
- sheet Diode_Bridge ports: added GND, Vin; removed none
Changed lines of the file:
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@@
 	(paper "A4")
 	(sheet
+		(at 107.95 132.08)
+		(size 54.61 26.67)
+		(exclude_from_sim no)
+		(in_bom yes)
+		(on_board yes)
+		(dnp no)
+		(fields_autoplaced yes)
+		(stroke
+			(width 0.1524)
+			(type solid)
+		)
+		(fill
+			(color 0 0 0 0)
+		)
+		(property "Sheetname" "UCC_Chip"
+			(at 107.95 131.3684 0)
+			(show_name no)
+			(do_not_autoplace no)
+			(effects
+				(font
+					(size 1.27 1.27)
+				)
+				(justify left bottom)
+			)
+		)
+		(property "Sheetfile" "UCC_Chip.kicad_sch"
+			(at 107.95 159.3346 0)
+			(hide yes)
+			(show_name no)
+			(do_not_autoplace no)
+			(effects
+				(font
+					(size 1.27 1.27)
+				)
+				(justify left top)
+			)
+		)
+		(instances
+			(project "Solar_Battery"
+				(path "/6805959e-39bb-4644-b93e-3970e29fedc0/a320594e-eb17-43a9-8193-2f75b3718179"
+					(page "6")
+				)
+			)
+		)
+	)
+	(sheet
 		(at 107.95 105.41)
-		(size 22.86 22.86)
+		(size 25.4 22.86)
 		(exclude_from_sim no)
 		(in_bom yes)
@@
 			)
 		)
+		(pin "GND" input
+			(at 107.95 116.84 180)
+			(effects
+				(font
+					(size 1.27 1.27)
+				)
+				(justify left)
+			)
+		)
+		(pin "Vin" input
+			(at 107.95 109.22 180)
+			(effects
+				(font
+					(size 1.27 1.27)
+				)
+				(justify left)
+			)
+		)
 		(instances
 			(project "Solar_Battery"
@@
 				)
 			)
+		)
+	)
+	(sheet
+		(at 138.43 105.41)
+		(size 24.13 22.86)
+		(exclude_from_sim no)
+		(in_bom yes)
+		(on_board yes)
+		(dnp no)
+		(fields_autoplaced yes)
+		(stroke
+			(width 0.1524)
+			(type solid)
+		)
+		(fill
+			(color 0 0 0 0)
+		)
+		(property "Sheetname" "Transformer_Output"
+			(at 138.43 104.6984 0)
+			(show_name no)
+			(do_not_autoplace no)
+			(effects
+				(font
+					(size 1.27 1.27)
+				)
+				(justify left bottom)
+			)
+		)
+		(property "Sheetfile" "Transformer_Output.kicad_sch"
+			(at 138.43 128.8546 0)
+			(hide yes)
+			(show_name no)
+			(do_not_autoplace no)
+			(effects
+				(font
+					(size 1.27 1.27)
+				)
+				(justify left top)
+			)
+		)
+		(instances
+			(project "Solar_Battery"
+				(path "/6805959e-39bb-4644-b93e-3970e29fedc0/a320594e-eb17-43a9-8193-2f75b3718179"
+					(page "5")
+				)
+			)

Commit message: misc
Other:
- sheet Diode_Bridge ports: added Iout; removed none
Changed lines of the file:
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@@
+			)
+		)
+		(pin "Iout" input
+			(at 133.35 114.3 0)
+			(effects
+				(font
+					(size 1.27 1.27)
+				)
+				(justify right)
 			)
 		)

Commit message: video2
Changed lines of the file:
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@@
 		)
 		(pin "GND" input
-			(at 107.95 116.84 180)
+			(at 107.95 120.65 180)
 			(effects
 				(font
@@
 		)
 		(pin "Vin" input
-			(at 107.95 109.22 180)
+			(at 107.95 113.03 180)
 			(effects
 				(font
@@
 		)
 		(pin "Iout" input
-			(at 133.35 114.3 0)
+			(at 133.35 115.57 0)
 			(effects
 				(font

Commit message: Changed Name of sheet
Other:
- sheet Diode_Bridge renamed Rectifier_Bridge
Changed lines of the file:
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@@
 			(color 0 0 0 0)
 		)
-		(property "Sheetname" "Diode_Bridge"
+		(property "Sheetname" "Rectifier_Bridge"
 			(at 107.95 104.6984 0)
 			(show_name no)

Commit message: note
Other:
- sheet Rectifier_Bridge renamed Rectifier_bridge
Changed lines of the file:
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@@
 			(color 0 0 0 0)
 		)
-		(property "Sheetname" "Rectifier_Bridge"
+		(property "Sheetname" "Rectifier_bridge"
 			(at 107.95 104.6984 0)
 			(show_name no)

Commit message: test
Other:
- sheet Rectifier_bridge renamed Diode_Bridge
Changed lines of the file:
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@@
 			(color 0 0 0 0)
 		)
-		(property "Sheetname" "Rectifier_bridge"
+		(property "Sheetname" "Diode_Bridge"
 			(at 107.95 104.6984 0)
 			(show_name no)
