File: Transformer_Output.kicad_sch (KiCad schematic)
At the start: 8 parts, among them T1 T1

Commit message: FixedMostIssues
Parts:
- C1+1: renamed from C1+; footprint Package_SON:Texas_DSG0008A_WSON-8-1EP_2x2mm_P0.5mm_EP0.9x1.6mm -> Capacitor_THT:C_Disc_D5.0mm_W2.5mm_P2.50mm
- CSNUB1: renamed from CSNUB; footprint (none) -> Capacitor_THT:C_Disc_D5.0mm_W2.5mm_P2.50mm
- renumbered + to +1, + to +2, + to +3, + to +4, + to +5
Changed lines of the file:
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@@
 		(dnp no)
 		(fields_autoplaced yes)
-		(property "Reference" "#PWR01"
+		(property "Reference" "#PWR015"
 			(at 119.38 106.68 0)
 			(hide yes)
@@
 			(project "Solar_Battery"
 				(path "/6805959e-39bb-4644-b93e-3970e29fedc0/a320594e-eb17-43a9-8193-2f75b3718179/7e488579-baf6-4b9f-affb-a6601b6eb832"
-					(reference "#PWR01")
+					(reference "#PWR015")
 					(unit 1)
 				)
@@
 		(in_pos_files yes)
 		(dnp no)
-		(property "Reference" "+"
+		(property "Reference" "+2"
 			(at 91.44 86.106 0)
 			(show_name no)
@@
 			(project "Solar_Battery"
 				(path "/6805959e-39bb-4644-b93e-3970e29fedc0/a320594e-eb17-43a9-8193-2f75b3718179/7e488579-baf6-4b9f-affb-a6601b6eb832"
-					(reference "+")
+					(reference "+2")
 					(unit 1)
 				)
@@
 		(in_pos_files yes)
 		(dnp no)
-		(property "Reference" "C1+"
+		(property "Reference" "C1+1"
 			(at 212.09 88.8999 90)
 			(show_name no)
@@
 			)
 		)
-		(property "Footprint" "Package_SON:Texas_DSG0008A_WSON-8-1EP_2x2mm_P0.5mm_EP0.9x1.6mm"
+		(property "Footprint" "Capacitor_THT:C_Disc_D5.0mm_W2.5mm_P2.50mm"
 			(at 209.2452 93.98 0)
 			(hide yes)
@@
 			(project "Solar_Battery"
 				(path "/6805959e-39bb-4644-b93e-3970e29fedc0/a320594e-eb17-43a9-8193-2f75b3718179/7e488579-baf6-4b9f-affb-a6601b6eb832"
-					(reference "C1+")
+					(reference "C1+1")
 					(unit 1)
 				)
@@
 		(in_pos_files yes)
 		(dnp no)
-		(property "Reference" "CSNUB"
+		(property "Reference" "CSNUB1"
 			(at 84.328 55.118 0)
 			(show_name no)
@@
 			)
 		)
-		(property "Footprint" ""
+		(property "Footprint" "Capacitor_THT:C_Disc_D5.0mm_W2.5mm_P2.50mm"
 			(at 94.9452 59.69 0)
 			(hide yes)
@@
 			(project "Solar_Battery"
 				(path "/6805959e-39bb-4644-b93e-3970e29fedc0/a320594e-eb17-43a9-8193-2f75b3718179/7e488579-baf6-4b9f-affb-a6601b6eb832"
-					(reference "CSNUB")
+					(reference "CSNUB1")
 					(unit 1)
 				)
@@
 		(in_pos_files yes)
 		(dnp no)
-		(property "Reference" "+"
+		(property "Reference" "+5"
 			(at 185.674 85.852 0)
 			(show_name no)
@@
 			(project "Solar_Battery"
 				(path "/6805959e-39bb-4644-b93e-3970e29fedc0/a320594e-eb17-43a9-8193-2f75b3718179/7e488579-baf6-4b9f-affb-a6601b6eb832"
-					(reference "+")
+					(reference "+5")
 					(unit 1)
 				)
@@
 		(in_pos_files yes)
 		(dnp no)
-		(property "Reference" "+"
+		(property "Reference" "+1"
 			(at 104.394 75.692 0)
 			(show_name no)
@@
 			(project "Solar_Battery"
 				(path "/6805959e-39bb-4644-b93e-3970e29fedc0/a320594e-eb17-43a9-8193-2f75b3718179/7e488579-baf6-4b9f-affb-a6601b6eb832"
-					(reference "+")
+					(reference "+1")
 					(unit 1)
 				)
@@
 		(in_pos_files yes)
 		(dnp no)
-		(property "Reference" "+"
+		(property "Reference" "+4"
 			(at 159.258 70.866 0)
 			(show_name no)
@@
 			(project "Solar_Battery"
 				(path "/6805959e-39bb-4644-b93e-3970e29fedc0/a320594e-eb17-43a9-8193-2f75b3718179/7e488579-baf6-4b9f-affb-a6601b6eb832"
-					(reference "+")
+					(reference "+4")
 					(unit 1)
 				)
@@
 		(in_pos_files yes)
 		(dnp no)
-		(property "Reference" "+"
+		(property "Reference" "+3"
 			(at 123.444 55.372 0)
 			(show_name no)
@@
 			(project "Solar_Battery"
 				(path "/6805959e-39bb-4644-b93e-3970e29fedc0/a320594e-eb17-43a9-8193-2f75b3718179/7e488579-baf6-4b9f-affb-a6601b6eb832"
-					(reference "+")
-					(unit 1)
-				)
+					(reference "+3")
+					(unit 1)
+				)

Commit message: PCB setup for next meeting
Parts:
- T1: footprint (none) -> Transformer_THT:Transformer_Toroid_Tapped_Horizontal_D10.5mm_Amidon-T37
Changed lines of the file:
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@@
 			)
 		)
-		(property "Footprint" ""
+		(property "Footprint" "Transformer_THT:Transformer_Toroid_Tapped_Horizontal_D10.5mm_Amidon-T37"
 			(at 146.05 83.82 0)
 			(hide yes)
