File: Battery_Controller.kicad_sch (KiCad schematic)
At the start: 0 parts

Commit message: video2
Other:
- added sheet c (Capacitor.kicad_sch)
Changed lines of the file:
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@@
 	(generator_version "10.0")
 	(paper "A4")
+	(sheet
+		(at 85.725 64.135)
+		(size 38.735 30.48)
+		(exclude_from_sim no)
+		(in_bom yes)
+		(on_board yes)
+		(dnp no)
+		(fields_autoplaced yes)
+		(stroke
+			(width 0.1524)
+			(type solid)
+		)
+		(fill
+			(color 0 0 0 0)
+		)
+		(property "Sheetname" "c"
+			(at 85.725 63.4234 0)
+			(show_name yes)
+			(do_not_autoplace no)
+			(effects
+				(font
+					(size 1.27 1.27)
+				)
+				(justify left bottom)
+			)
+		)
+		(property "Sheetfile" "Capacitor.kicad_sch"
+			(at 85.725 95.1996 0)
+			(show_name no)
+			(do_not_autoplace no)
+			(effects
+				(font
+					(size 1.27 1.27)
+				)
+				(justify left top)
+			)
+		)
+		(instances
+			(project "Solar_Battery"
+				(path "/6805959e-39bb-4644-b93e-3970e29fedc0/49420c5f-19b8-4027-9796-8766afa78876"
+					(page "7")
+				)
+			)
+		)
+	)
 )

Commit message: deleted extra sheet
Other:
- removed sheet c
Changed lines of the file:
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@@
 	(generator_version "10.0")
 	(paper "A4")
-	(sheet
-		(at 85.725 64.135)
-		(size 38.735 30.48)
-		(exclude_from_sim no)
-		(in_bom yes)
-		(on_board yes)
-		(dnp no)
-		(fields_autoplaced yes)
-		(stroke
-			(width 0.1524)
-			(type solid)
-		)
-		(fill
-			(color 0 0 0 0)
-		)
-		(property "Sheetname" "c"
-			(at 85.725 63.4234 0)
-			(show_name yes)
-			(do_not_autoplace no)
-			(effects
-				(font
-					(size 1.27 1.27)
-				)
-				(justify left bottom)
-			)
-		)
-		(property "Sheetfile" "Capacitor.kicad_sch"
-			(at 85.725 95.1996 0)
-			(show_name no)
-			(do_not_autoplace no)
-			(effects
-				(font
-					(size 1.27 1.27)
-				)
-				(justify left top)
-			)
-		)
-		(instances
-			(project "Solar_Battery"
-				(path "/6805959e-39bb-4644-b93e-3970e29fedc0/49420c5f-19b8-4027-9796-8766afa78876"
-					(page "7")
-				)
-			)
-		)
-	)
 )
