File: Battery_Controller.kicad_sch (KiCad schematic)
At the start: 20 parts, among them SW1 SW_Push, U1 BQ25895RTWR

Commit message: FixedMostIssues
Parts:
- C1: renamed from C2; footprint Package_SO:SOIC-8_3.9x4.9mm_P1.27mm -> Capacitor_THT:C_Disc_D5.0mm_W2.5mm_P2.50mm
- C2: renamed from C1; footprint (none) -> Capacitor_THT:C_Disc_D5.0mm_W2.5mm_P2.50mm
- C3: renamed from C5; footprint Package_SO:SOIC-8_3.9x4.9mm_P1.27mm -> Capacitor_THT:C_Disc_D5.0mm_W2.5mm_P2.50mm
- C4: renamed from C8; footprint (none) -> Capacitor_THT:C_Disc_D5.0mm_W2.5mm_P2.50mm
- C5: renamed from C6; footprint Package_SO:SOIC-8_3.9x4.9mm_P1.27mm -> Capacitor_THT:C_Disc_D5.0mm_W2.5mm_P2.50mm
- C6: renamed from C7; footprint Package_SO:SOIC-8_3.9x4.9mm_P1.27mm -> Capacitor_THT:C_Disc_D5.0mm_W2.5mm_P2.50mm
- C7: renamed from C9; footprint (none) -> Capacitor_THT:C_Disc_D5.0mm_W2.5mm_P2.50mm
- R1: renamed from R3; footprint (none) -> Resistor_THT:R_Axial_DIN0207_L6.3mm_D2.5mm_P10.16mm_Horizontal
- R2: renamed from R4; footprint (none) -> Resistor_THT:R_Axial_DIN0207_L6.3mm_D2.5mm_P10.16mm_Horizontal
- R3: renamed from R5; footprint (none) -> Resistor_THT:R_Axial_DIN0207_L6.3mm_D2.5mm_P10.16mm_Horizontal
- R4: renamed from R1; footprint (none) -> Resistor_THT:R_Axial_DIN0207_L6.3mm_D2.5mm_P10.16mm_Horizontal
- R5: renamed from R2; footprint (none) -> Resistor_THT:R_Axial_DIN0207_L6.3mm_D2.5mm_P10.16mm_Horizontal
- R6, R7: footprint Package_DIP:DIP-8_W7.62mm -> Resistor_THT:R_Axial_DIN0207_L6.3mm_D2.5mm_P10.16mm_Horizontal
- R8: footprint (none) -> Resistor_THT:R_Axial_DIN0207_L6.3mm_D2.5mm_P10.16mm_Horizontal
- renumbered D5 to D1, L2 to L1

Commit message: Started PCB
Parts:
- removed BT1: Battery_Cell, Package_SO:SOIC-20W_7.5x12.8mm_P1.27mm, symbol Device:Battery_Cell
- removed C1: 40µF, Capacitor_THT:C_Disc_D5.0mm_W2.5mm_P2.50mm, symbol Device:C_Small
- removed C2: 1µF, Capacitor_THT:C_Disc_D5.0mm_W2.5mm_P2.50mm, symbol Device:C_Small
- removed C3: 47nF, Capacitor_THT:C_Disc_D5.0mm_W2.5mm_P2.50mm, symbol Device:C_Small
- removed C4: 4.7µF, Capacitor_THT:C_Disc_D5.0mm_W2.5mm_P2.50mm, symbol Device:C_Small
- removed C5, C6: 10µF, Capacitor_THT:C_Disc_D5.0mm_W2.5mm_P2.50mm, symbol Device:C_Small
- removed C7: 10uF, Capacitor_THT:C_Disc_D5.0mm_W2.5mm_P2.50mm, symbol Device:C_Small
- removed D1: LED_1, OptoDevice:R_LDR_D6.4mm_P3.4mm_Vertical, symbol Device:LED_Small_Filled
- removed L1: 2.2µH, Inductor_SMD:L_CommonModeChoke_Coilcraft_0603USB, symbol Device:L_Small
- removed R1, R2, R3: 10kΩ, Resistor_THT:R_Axial_DIN0207_L6.3mm_D2.5mm_P10.16mm_Horizontal, symbol Device:R_Small_US
- removed R4: 260Ω, Resistor_THT:R_Axial_DIN0207_L6.3mm_D2.5mm_P10.16mm_Horizontal, symbol Device:R_Small_US
- removed R5: 2.2KΩ, Resistor_THT:R_Axial_DIN0207_L6.3mm_D2.5mm_P10.16mm_Horizontal, symbol Device:R_Small_US
- removed R6: 5.23KΩ, Resistor_THT:R_Axial_DIN0207_L6.3mm_D2.5mm_P10.16mm_Horizontal, symbol Device:R_Small_US
- removed R7: 30.1KΩ, Resistor_THT:R_Axial_DIN0207_L6.3mm_D2.5mm_P10.16mm_Horizontal, symbol Device:R_Small_US
- removed R8: 10KΩ, Resistor_THT:R_Axial_DIN0207_L6.3mm_D2.5mm_P10.16mm_Horizontal, symbol Device:R_Small_US
- removed SW1: SW_Push, Button_Switch_SMD:SW_SPST_CK_KMS2xxGP, symbol Switch:SW_Push
- removed U1: BQ25895RTWR, BQ:RTW0024H, symbol BQ:BQ25895RTWR
Other:
- note removed: "3 Humps in Diagram"
- note removed: "Circles should be completely black"
- note removed: "Treating it as /CE"
