File: UCC_Chip.kicad_sch (KiCad schematic)
At the start: 10 parts

Commit message: NewUCCschem
Parts:
- added U2: UCC28710DR, SO_UCC28710D_TEX, symbol UCCfixed:UCC28710DR
Connections:
- net GND: now also U2.4 (GND)
- net at +.1 (K), +.2, CDD.1: now also U2.1 (VDD)
- net at +.1: now also U2.5 (CS)
Other:
- moved on the sheet: +, CDD

Commit message: UCC_Chip_Final
Connections:
- net Rectifier_UCC_In: now also U2.8 (HV)
Changed lines of the file:
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@@
 	(hierarchical_label "Rectifier_UCC_In"
 		(shape input)
-		(at 121.92 45.72 0)
+		(at 132.08 92.71 0)
 		(effects
 			(font
