File: Diode_Bridge.kicad_sch (KiCad schematic)
At the start: 8 parts

Commit message: Added the ucc28710 symbol in the schematic and its footprint. Added the mosfet symbol. Connected the final missing connections in the schematics. annotated  it. if done right, only a few footprints need assignment in the uccchip subsheet
Parts:
- renumbered Cin to Cin1, Dac to Dac1, Dac to Dac2, Dac to Dac3, Dac to Dac4, Rl to Rl1
Changed lines of the file:
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@@
+				)
+			)
+			(project "Rectifier"
+				(path "/fabf5a3f-f60f-4bcb-816d-2ffdd48e9531/66c5df4f-46ad-4d4f-997c-052ec03a6539"
+					(reference "Cin2")
+					(unit 1)
 				)
 			)
@@
 				)
 			)
+			(project "Rectifier"
+				(path "/fabf5a3f-f60f-4bcb-816d-2ffdd48e9531/66c5df4f-46ad-4d4f-997c-052ec03a6539"
+					(reference "L1")
+					(unit 1)
+				)
+			)
 		)
 	)
@@
 		(dnp no)
 		(fields_autoplaced yes)
-		(property "Reference" "Rl"
+		(property "Reference" "Rl1"
 			(at 101.6 60.96 90)
 			(show_name no)
@@
 				(path "/6805959e-39bb-4644-b93e-3970e29fedc0/a320594e-eb17-43a9-8193-2f75b3718179/66c5df4f-46ad-4d4f-997c-052ec03a6539"
 					(reference "Rl")
+					(unit 1)
+				)
+			)
+			(project "Rectifier"
+				(path "/fabf5a3f-f60f-4bcb-816d-2ffdd48e9531/66c5df4f-46ad-4d4f-997c-052ec03a6539"
+					(reference "Rl1")
 					(unit 1)
 				)
@@
 				)
 			)
+			(project "Rectifier"
+				(path "/fabf5a3f-f60f-4bcb-816d-2ffdd48e9531/66c5df4f-46ad-4d4f-997c-052ec03a6539"
+					(reference "#PWR02")
+					(unit 1)
+				)
+			)
 		)
 	)
@@
 		(dnp no)
 		(fields_autoplaced yes)
-		(property "Reference" "Dac"
+		(property "Reference" "Dac2"
 			(at 123.19 78.74 0)
 			(show_name no)
@@
 				(path "/6805959e-39bb-4644-b93e-3970e29fedc0/a320594e-eb17-43a9-8193-2f75b3718179/66c5df4f-46ad-4d4f-997c-052ec03a6539"
 					(reference "Dac")
+					(unit 1)
+				)
+			)
+			(project "Rectifier"
+				(path "/fabf5a3f-f60f-4bcb-816d-2ffdd48e9531/66c5df4f-46ad-4d4f-997c-052ec03a6539"
+					(reference "Dac2")
 					(unit 1)
 				)
@@
 		(dnp no)
 		(fields_autoplaced yes)
-		(property "Reference" "Dac"
+		(property "Reference" "Dac3"
 			(at 133.35 68.58 0)
 			(show_name no)
@@
 				(path "/6805959e-39bb-4644-b93e-3970e29fedc0/a320594e-eb17-43a9-8193-2f75b3718179/66c5df4f-46ad-4d4f-997c-052ec03a6539"
 					(reference "Dac")
+					(unit 1)
+				)
+			)
+			(project "Rectifier"
+				(path "/fabf5a3f-f60f-4bcb-816d-2ffdd48e9531/66c5df4f-46ad-4d4f-997c-052ec03a6539"
+					(reference "Dac3")
 					(unit 1)
 				)
@@
 		(dnp no)
 		(fields_autoplaced yes)
-		(property "Reference" "Dac"
+		(property "Reference" "Dac4"
 			(at 133.35 78.74 0)
 			(show_name no)
@@
 				(path "/6805959e-39bb-4644-b93e-3970e29fedc0/a320594e-eb17-43a9-8193-2f75b3718179/66c5df4f-46ad-4d4f-997c-052ec03a6539"
 					(reference "Dac")
+					(unit 1)
+				)
+			)
+			(project "Rectifier"
+				(path "/fabf5a3f-f60f-4bcb-816d-2ffdd48e9531/66c5df4f-46ad-4d4f-997c-052ec03a6539"
+					(reference "Dac4")
 					(unit 1)
 				)
@@
 		(dnp no)
 		(fields_autoplaced yes)
-		(property "Reference" "#PWR03"
+		(property "Reference" "#PWR01"
 			(at 127 99.06 0)
 			(hide yes)
@@
 				(path "/6805959e-39bb-4644-b93e-3970e29fedc0/a320594e-eb17-43a9-8193-2f75b3718179/66c5df4f-46ad-4d4f-997c-052ec03a6539"
 					(reference "#PWR03")
+					(unit 1)
+				)
+			)
+			(project "Rectifier"
+				(path "/fabf5a3f-f60f-4bcb-816d-2ffdd48e9531/66c5df4f-46ad-4d4f-997c-052ec03a6539"
+					(reference "#PWR01")
 					(unit 1)
 				)
@@
 		(dnp no)
 		(fields_autoplaced yes)
-		(property "Reference" "Dac"
+		(property "Reference" "Dac1"
 			(at 120.65 68.58 0)
 			(show_name no)
@@
 				(path "/6805959e-39bb-4644-b93e-3970e29fedc0/a320594e-eb17-43a9-8193-2f75b3718179/66c5df4f-46ad-4d4f-997c-052ec03a6539"
 					(reference "Dac")
+					(unit 1)
+				)
+			)
+			(project "Rectifier"
+				(path "/fabf5a3f-f60f-4bcb-816d-2ffdd48e9531/66c5df4f-46ad-4d4f-997c-052ec03a6539"
+					(reference "Dac1")
 					(unit 1)
 				)
@@
 		(dnp no)
 		(fields_autoplaced yes)
-		(property "Reference" "Cin"
+		(property "Reference" "Cin1"
 			(at 156.21 78.7399 0)
 			(show_name no)
@@
 					(unit 1)
 				)
+			)
+			(project "Rectifier"
+				(path "/fabf5a3f-f60f-4bcb-816d-2ffdd48e9531/66c5df4f-46ad-4d4f-997c-052ec03a6539"
+					(reference "Cin1")
+					(unit 1)
+				)
