File: Solar_Battery.kicad_pcb (KiCad board)
At the start: 2 copper layers, 49 parts, among them SW1 SW_Push, T1 T1, U1 BQ25895RTWR, U1 UCC28710DR, U2 IRF830APBF, U3 UCC28710DR

Commit message: Started PCB
Parts:
- removed BT1: Battery_Cell, Package_SO:SOIC-20W_7.5x12.8mm_P1.27mm
- removed U1: BQ25895RTWR, BQ:RTW0024H
- removed U1: UCC28710DR, ucc:SO_UCC28710D_TEX
- moved CSNUB1 79.8 mm to (110.5, 31.0)
- moved Dac1 77.7 mm to (31.3, 115.0)
- moved +2 71.6 mm to (185.9, 59.5)
- moved U3 63.6 mm to (73.5, 80.0)
- moved CDD1 60.6 mm to (77.5, 61.5)
- moved +1 37.0 mm to (139.2, 44.5)
- moved +3 37.0 mm to (119.2, 44.0)
- moved T1 36.6 mm to (217.0, 78.7)
- moved SW1 10.9 mm to (33.0, 21.0)
- moved L1 10.0 mm to (30.5, 30.5)
- moved Dac2 0.23 mm to (30.8, 43.0)
Connections:
- +10 pad 2: Earth -> GND
- +13 pad 1: Earth -> GND
- +6 pad 1: Earth -> GND
- +9 pad 2: Earth -> GND
- CDD1 pad 2: Earth -> GND
- Cin1 pad 2: Earth -> GND
- Cin2 pad 2: Earth -> GND
- Dac2 pad 2: Earth -> GND
- Dac4 pad 2: Earth -> GND
- T1 pad 5: Earth -> GND
- U3 pad 4: Earth -> GND
Other:
- board text added: "Transformer Node 1"
