File: Solar_Battery.kicad_pcb (KiCad board)
At the start: 2 copper layers, 49 parts, among them SW1 SW_Push, T1 T1, U1 BQ25895RTWR, U1 UCC28710DR, U2 IRF830APBF, U3 UCC28710DR

Commit message: PCBstartedJuan
Parts:
- removed BT1: Battery_Cell, Package_SO:SOIC-20W_7.5x12.8mm_P1.27mm
- removed C1: 40µF, Capacitor_THT:C_Disc_D5.0mm_W2.5mm_P2.50mm
- removed C2: 1µF, Capacitor_THT:C_Disc_D5.0mm_W2.5mm_P2.50mm
- removed C3: 47nF, Capacitor_THT:C_Disc_D5.0mm_W2.5mm_P2.50mm
- removed C4: 4.7µF, Capacitor_THT:C_Disc_D5.0mm_W2.5mm_P2.50mm
- removed C5, C6: 10µF, Capacitor_THT:C_Disc_D5.0mm_W2.5mm_P2.50mm
- removed C7: 10uF, Capacitor_THT:C_Disc_D5.0mm_W2.5mm_P2.50mm
- removed D1: LED_1, OptoDevice:R_LDR_D6.4mm_P3.4mm_Vertical
- removed L1: 2.2µH, Inductor_SMD:L_CommonModeChoke_Coilcraft_0603USB
- removed R1, R2, R3: 10kΩ, Resistor_THT:R_Axial_DIN0207_L6.3mm_D2.5mm_P10.16mm_Horizontal
- removed R4: 260Ω, Resistor_THT:R_Axial_DIN0207_L6.3mm_D2.5mm_P10.16mm_Horizontal
- removed R5: 2.2KΩ, Resistor_THT:R_Axial_DIN0207_L6.3mm_D2.5mm_P10.16mm_Horizontal
- removed R6: 5.23KΩ, Resistor_THT:R_Axial_DIN0207_L6.3mm_D2.5mm_P10.16mm_Horizontal
- removed R7: 30.1KΩ, Resistor_THT:R_Axial_DIN0207_L6.3mm_D2.5mm_P10.16mm_Horizontal
- removed R8: 10KΩ, Resistor_THT:R_Axial_DIN0207_L6.3mm_D2.5mm_P10.16mm_Horizontal
- removed SW1: SW_Push, Button_Switch_SMD:SW_SPST_CK_KMS2xxGP
- removed U1: BQ25895RTWR, BQ:RTW0024H
- removed U1: UCC28710DR, ucc:SO_UCC28710D_TEX
- moved U3 109.9 mm to (118.5, 93.0)
- moved CDD1 83.3 mm to (90.3, 96.8)
- moved +10 83.3 mm to (87.7, 81.5)
- moved +11 83.3 mm to (74.4, 91.6)
- moved +12 83.3 mm to (87.7, 85.0)
- moved +13 83.3 mm to (74.4, 95.7)
- moved +14 83.3 mm to (74.4, 99.7)
- moved +7 83.3 mm to (74.4, 79.5)
- moved +8 83.3 mm to (74.4, 83.5)
- moved +9 83.3 mm to (74.4, 87.5)
- moved U2 83.3 mm to (91.3, 76.5)
- moved +6 78.4 mm to (77.9, 51.5)
- moved CSNUB1 71.8 mm to (104.0, 25.5)
- moved Cin2 71.0 mm to (92.5, 25.0), turned to -90 degrees
- moved Cin1 52.4 mm to (73.0, 25.5), turned to -90 degrees
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Connections:
- net Earth renamed GND
